Commit message: real HW - beta2

File: xarm_description/urdf/xarm7.urdf.xacro (robot description, xacro)
@@ -7,9 +7,9 @@
   <xacro:macro name="xarm7_urdf" params="prefix
     joint1_lower_limit:=${-2.0*pi}  joint1_upper_limit:=${2.0*pi}
-    joint2_lower_limit:=${-2.0*pi}  joint2_upper_limit:=${2.0*pi}
+    joint2_lower_limit:=${-2.18}  joint2_upper_limit:=${2.18}
     joint3_lower_limit:=${-2.0*pi}  joint3_upper_limit:=${2.0*pi}
-    joint4_lower_limit:=${-2.0*pi}  joint4_upper_limit:=${2.0*pi}
+    joint4_lower_limit:=${-4.01}  joint4_upper_limit:=${0.11}
     joint5_lower_limit:=${-2.0*pi}  joint5_upper_limit:=${2.0*pi}
-    joint6_lower_limit:=${-2.0*pi}  joint6_upper_limit:=${2.0*pi}
+    joint6_lower_limit:=${-1.75}  joint6_upper_limit:=${1.0*pi}
     joint7_lower_limit:=${-2.0*pi}  joint7_upper_limit:=${2.0*pi}">
     <material name="Black">
@@ -230,5 +230,5 @@
       <child link="${prefix}link5"/>
       <origin xyz="0.0785 0 -0.336" rpy="0 0 0"/>
-      <axis xyz="0 0 1"/>
+      <axis xyz="0 0 -1"/>
       <limit
         lower="${joint5_lower_limit}"
@@ -306,5 +306,5 @@
       <child link="${prefix}link7"/>
       <origin xyz="0.073 0 -0.0695" rpy="0 0 0"/>
-      <axis xyz="0 0 1"/>
+      <axis xyz="0 0 -1"/>
       <limit
         lower="${joint7_lower_limit}"
