Commit message: small optimizations

File: xarm_description/urdf/xarm6.urdf.xacro (robot description, xacro)
@@ -52,5 +52,5 @@
           <mesh filename="package://xarm_description/meshes/xarm6/visual/link1.stl"/>
         </geometry>
-        <origin xyz="0 0 -0.2655" rpy="0 0 0"/>
+        <origin xyz="0 0 -0.267" rpy="0 0 0"/>
         <material name="White" />
       </visual>
@@ -59,5 +59,5 @@
           <mesh filename="package://xarm_description/meshes/xarm6/visual/link1.stl"/>
         </geometry>
-        <origin xyz="0 0 -0.2655" rpy="0 0 0"/>
+        <origin xyz="0 0 -0.267" rpy="0 0 0"/>
       </collision>
       <inertial>
@@ -76,5 +76,5 @@
       <parent link="${prefix}link_base"/>
       <child  link="${prefix}link1"/>
-      <origin xyz="0 0 0.2655" rpy="0 0 0"/>
+      <origin xyz="0 0 0.267" rpy="0 0 0"/>
       <axis   xyz="0 0 1"/>
       <limit
@@ -90,5 +90,5 @@
           <mesh filename="package://xarm_description/meshes/xarm6/visual/link2.stl"/>
         </geometry>
-        <origin xyz="0 0 -0.2655" rpy="0 0 0"/>
+        <origin xyz="0 0 -0.267" rpy="0 0 0"/>
         <material name="White" />
       </visual>
@@ -97,5 +97,5 @@
           <mesh filename="package://xarm_description/meshes/xarm6/visual/link2.stl"/>
         </geometry>
-        <origin xyz="0 0 -0.2655" rpy="0 0 0"/>
+        <origin xyz="0 0 -0.267" rpy="0 0 0"/>
       </collision>
       <inertial>
